Commit message: update 2026-06-23 23:47:54

File: ros_motion_planning/src/sim_env/urdf/my_car/my_car.urdf (robot description, URDF)
Before this commit: robot my_car, 7 links, 6 joints
Joints:
- joint base_scan_joint: origin xyz=-0.00074 0.187 0.076 rpy=0 0 0 -> xyz=-0.00074 0.187 -0.076 rpy=0 0 0
- joint left_wheel_front_joint: origin xyz=-0.104 5.3E-05 0.085 rpy=0 0 0 -> xyz=-0.104 5.3E-05 -0.085 rpy=0 0 0
- joint left_wheel_rear_joint: origin xyz=-0.104 4.0E-05 0.421 rpy=0 0 0 -> xyz=-0.104 4.0E-05 -0.421 rpy=0 0 0
- joint right_wheel_front_joint: origin xyz=0.104 -4.1E-05 0.087 rpy=0 0 0 -> xyz=0.104 -4.1E-05 -0.087 rpy=0 0 0
- joint right_wheel_rear_joint: origin xyz=0.104 0.00056 0.423 rpy=0 0 0 -> xyz=0.104 0.00056 -0.423 rpy=0 0 0

Commit message: update 2026-06-24 12:22:59

File: ros_motion_planning/src/sim_env/urdf/my_car/my_car.urdf (robot description, URDF)
Before this commit: robot my_car, 7 links, 6 joints
Joints:
- joint base_footprint_joint: origin xyz=0 0 0 rpy=1.5708 0 1.5708 -> xyz=0 0 0 rpy=1.5708 0 -1.5708
- joint base_scan_joint: origin xyz=-0.00074 0.187 -0.076 rpy=0 0 0 -> xyz=-0.00074 0.187 0.076 rpy=0 0 0
- joint left_wheel_front_joint: origin xyz=-0.104 5.3E-05 -0.085 rpy=0 0 0 -> xyz=-0.104 5.3E-05 0.085 rpy=0 0 0
- joint left_wheel_rear_joint: origin xyz=-0.104 4.0E-05 -0.421 rpy=0 0 0 -> xyz=-0.104 4.0E-05 0.421 rpy=0 0 0
- joint right_wheel_front_joint: origin xyz=0.104 -4.1E-05 -0.087 rpy=0 0 0 -> xyz=0.104 -4.1E-05 0.087 rpy=0 0 0
- joint right_wheel_rear_joint: origin xyz=0.104 0.00056 -0.423 rpy=0 0 0 -> xyz=0.104 0.00056 0.423 rpy=0 0 0

Commit message: update 2026-06-24 13:16:12

File: ros_motion_planning/src/sim_env/urdf/my_car/my_car.urdf (robot description, URDF)
Before this commit: robot my_car, 7 links, 6 joints
Joints:
- joint base_footprint_joint: origin xyz=0 0 0 rpy=1.5708 0 -1.5708 -> xyz=0 0 0.1105 rpy=1.5708 0 -1.5708
- joint left_wheel_front_joint: origin xyz=-0.104 5.3E-05 0.085 rpy=0 0 0 -> xyz=-0.104 -0.004 0.085 rpy=0 0 0
- joint left_wheel_rear_joint: origin xyz=-0.104 4.0E-05 0.421 rpy=0 0 0 -> xyz=-0.104 -0.004 0.421 rpy=0 0 0
- joint right_wheel_front_joint: origin xyz=0.104 -4.1E-05 0.087 rpy=0 0 0 -> xyz=0.104 -0.004 0.087 rpy=0 0 0
- joint right_wheel_rear_joint: origin xyz=0.104 0.00056 0.423 rpy=0 0 0 -> xyz=0.104 -0.004 0.423 rpy=0 0 0
