Commit message: update 2026-06-24 18:45:13

File: gazebo_create/urdf/my_car/my_car.urdf (robot description, URDF)
Before this commit: robot my_car, 7 links, 6 joints
Joints:
- joint base_footprint_joint: origin xyz=0 0 0.1105 rpy=1.5708 0 -1.5708 -> xyz=0 0 0.1105 rpy=1.5708 0 1.5708

Commit message: update 2026-06-24 19:00:50

File: gazebo_create/urdf/my_car/my_car.urdf (robot description, URDF)
Before this commit: robot my_car, 7 links, 6 joints
Joints:
- joint base_footprint_joint: origin xyz=0 0 0.1105 rpy=1.5708 0 1.5708 -> xyz=0 0 0.1105 rpy=1.5708 0 -1.5708

Commit message: update 2026-06-24 19:20:16

File: gazebo_create/urdf/my_car/my_car.urdf (robot description, URDF)
Before this commit: robot my_car, 7 links, 6 joints
Joints:
- joint base_footprint_joint: origin xyz=0 0 0.1105 rpy=1.5708 0 -1.5708 -> xyz=0 0 0.1105 rpy=0 0 0

Commit message: update 2026-06-24 19:25:10

File: gazebo_create/urdf/my_car/my_car.urdf (robot description, URDF)
Before this commit: robot my_car, 7 links, 6 joints
Joints:
- joint base_footprint_joint: origin xyz=0 0 0.1105 rpy=0 0 0 -> xyz=0 0 0.1105 rpy=1.5708 0 -1.5708

Commit message: update 2026-06-24 20:29:20

File: gazebo_create/urdf/my_car/my_car.urdf (robot description, URDF)
Before this commit: robot my_car, 7 links, 6 joints
Joints:
- joint base_scan_joint: origin xyz=-0.00074 0.187 0.076 rpy=0 0 0 -> xyz=-0.00074 0.187 -0.178 rpy=0 0 0
- joint left_wheel_front_joint: origin xyz=-0.104 -0.004 0.085 rpy=0 0 0 -> xyz=-0.104 -0.004 -0.169 rpy=0 0 0
- joint left_wheel_rear_joint: origin xyz=-0.104 -0.004 0.421 rpy=0 0 0 -> xyz=-0.104 -0.004 0.167 rpy=0 0 0
- joint right_wheel_front_joint: origin xyz=0.104 -0.004 0.087 rpy=0 0 0 -> xyz=0.104 -0.004 -0.167 rpy=0 0 0
- joint right_wheel_rear_joint: origin xyz=0.104 -0.004 0.423 rpy=0 0 0 -> xyz=0.104 -0.004 0.169 rpy=0 0 0

Commit message: update 2026-06-24 20:34:09

File: gazebo_create/urdf/my_car/my_car.urdf (robot description, URDF)
Before this commit: robot my_car, 7 links, 6 joints
Joints:
- joint base_footprint_joint: origin xyz=0 0 0.1105 rpy=1.5708 0 -1.5708 -> xyz=-0.254 0 0.1105 rpy=1.5708 0 -1.5708

Commit message: update 2026-06-24 21:09:03

File: gazebo_create/urdf/my_car/my_car.urdf (robot description, URDF)
Before this commit: robot my_car, 7 links, 6 joints
Joints:
- joint base_scan_joint: origin xyz=-0.00074 0.187 -0.178 rpy=0 0 0 -> xyz=-0.00074 0.127 -0.178 rpy=0 0 0

Commit message: update 2026-06-24 21:22:59

File: gazebo_create/urdf/my_car/my_car.urdf (robot description, URDF)
Before this commit: robot my_car, 7 links, 6 joints
Joints:
- joint base_footprint_joint: origin xyz=-0.254 0 0.1105 rpy=1.5708 0 -1.5708 -> xyz=-0.254 0 0.1105 rpy=1.5708 0 1.5708
- joint base_scan_joint: origin xyz=-0.00074 0.127 -0.178 rpy=0 0 0 -> xyz=0.00074 0.127 0.178 rpy=0 0 0
- joint left_wheel_front_joint: origin xyz=-0.104 -0.004 -0.169 rpy=0 0 0 -> xyz=0.104 -0.004 0.169 rpy=0 0 0
- joint left_wheel_rear_joint: origin xyz=-0.104 -0.004 0.167 rpy=0 0 0 -> xyz=0.104 -0.004 -0.167 rpy=0 0 0
- joint right_wheel_front_joint: origin xyz=0.104 -0.004 -0.167 rpy=0 0 0 -> xyz=-0.104 -0.004 0.167 rpy=0 0 0
- joint right_wheel_rear_joint: origin xyz=0.104 -0.004 0.169 rpy=0 0 0 -> xyz=-0.104 -0.004 -0.169 rpy=0 0 0

Commit message: update 2026-06-24 21:27:34

File: gazebo_create/urdf/my_car/my_car.urdf (robot description, URDF)
Before this commit: robot my_car, 7 links, 6 joints
Joints:
- joint base_footprint_joint: origin xyz=-0.254 0 0.1105 rpy=1.5708 0 1.5708 -> xyz=-0.254 0 0.1105 rpy=1.5708 0 -1.5708
- joint base_scan_joint: origin xyz=0.00074 0.127 0.178 rpy=0 0 0 -> xyz=-0.00074 0.127 -0.178 rpy=0 0 0
- joint left_wheel_front_joint: origin xyz=0.104 -0.004 0.169 rpy=0 0 0 -> xyz=-0.104 -0.004 -0.169 rpy=0 0 0
- joint left_wheel_rear_joint: origin xyz=0.104 -0.004 -0.167 rpy=0 0 0 -> xyz=-0.104 -0.004 0.167 rpy=0 0 0
- joint right_wheel_front_joint: origin xyz=-0.104 -0.004 0.167 rpy=0 0 0 -> xyz=0.104 -0.004 -0.167 rpy=0 0 0
- joint right_wheel_rear_joint: origin xyz=-0.104 -0.004 -0.169 rpy=0 0 0 -> xyz=0.104 -0.004 0.169 rpy=0 0 0

Commit message: update 2026-06-24 22:06:03

File: gazebo_create/urdf/my_car/my_car.urdf (robot description, URDF)
Before this commit: robot my_car, 7 links, 6 joints
Joints:
- joint base_scan_joint: origin xyz=-0.00074 0.127 -0.178 rpy=0 0 0 -> xyz=-0.00074 0.127 -0.178 rpy=-1.5708 0 0

Commit message: update 2026-06-24 22:15:38

File: gazebo_create/urdf/my_car/my_car.urdf (robot description, URDF)
Before this commit: robot my_car, 7 links, 6 joints
Joints:
- joint base_scan_joint: origin xyz=-0.00074 0.127 -0.178 rpy=-1.5708 0 0 -> xyz=-0.076 0.00074 0.2375 rpy=0 0 0; parent base_link -> base_footprint
