Commit message: update 2026-06-25 14:18:56

File: ros_motion_planning/my_robot/urdf/my_robot.urdf (robot description, URDF)
Before this commit: robot 1, 6 links, 5 joints
Links:
- link base_link: mass 3.6348 -> 3.63476292057873; geometry collision mesh filename=package://my_robot/meshes/base_link.STL; visual mesh filename=package://my_robot/meshes/base_link.STL
- link base_scan: mass 0 -> 0.0374307462908558; geometry collision mesh filename=package://my_robot/meshes/base_scan.STL; visual mesh filename=package://my_robot/meshes/base_scan.STL
- link left_wheel_front_Link: mass 0.82615 -> 0.826148513927948; geometry collision mesh filename=package://my_robot/meshes/left_wheel_front_Link.STL; visual mesh filename=package://my_robot/meshes/left_wheel_front_Link.STL
- link left_wheel_rear_Link: geometry collision mesh filename=package://my_robot/meshes/left_wheel_rear_Link.STL; visual mesh filename=package://my_robot/meshes/left_wheel_rear_Link.STL
- link right_wheel_front_Link: mass 0.826148517222633 -> 0.826148517222712; geometry collision mesh filename=package://my_robot/meshes/right_wheel_front_Link.STL; visual mesh filename=package://my_robot/meshes/right_wheel_front_Link.STL
- link right_wheel_rear_Link: mass 0.826148517020799 -> 0.826148517020798; geometry collision mesh filename=package://my_robot/meshes/right_wheel_rear_Link.STL; visual mesh filename=package://my_robot/meshes/right_wheel_rear_Link.STL
Joints:
- joint base_scan_joint: origin xyz=-0.000737150267890688 0.186848211076242 0.0757259001306266 rpy=0 0 0 -> xyz=0.190432245902798 0.00406027485239292 0.216848211077121 rpy=0 0 0
- joint left_wheel_front_joint: axis -0.99997 0.00045312 -0.0072447 -> -0.0102031718617054 0.999947843638991 0.000453084641131486; origin xyz=-0.1039 5.2752E-05 0.085448 rpy=0 0 0 -> xyz=0.178912109148856 0.107037805223412 0.030052752271374 rpy=0 0 0
- joint left_wheel_rear_joint: axis 0.99998 0.0024952 0.0060631 -> 0.0113846376579507 -0.999932079719297 0.00249519010073403; origin xyz=-0.1039 4.0099E-05 0.42145 rpy=0 0 0 -> xyz=-0.157035966824235 0.101175564800452 0.0300400994124252 rpy=0 0 0
- joint right_wheel_front_joint: axis -0.99997 0.00045312 -0.0072447 -> -0.0102031718617054 0.999947843638991 0.000453084641131486; origin xyz=0.1039 -4.1409E-05 0.086953 rpy=0 0 0 -> xyz=0.181032384121442 -0.10075683114026 0.0299585988024258 rpy=0 0 0
- joint right_wheel_rear_joint: axis 0.99998 0.0024952 0.0060631 -> 0.0113846376579507 -0.999932079719297 0.00249519010073403; origin xyz=0.1039 0.00055861 0.42271 rpy=0 0 0 -> xyz=-0.154670188269395 -0.106614787564809 0.0305586110601316 rpy=0 0 0

Commit message: update 2026-06-26 16:08:54

File: ros_motion_planning/my_robot/urdf/my_robot.urdf (robot description, URDF)
Before this commit: robot my_robot, 6 links, 5 joints
Links:
- link base_link: geometry visual mesh filename=package://my_robot/meshes/base_link.STL
- link base_scan: geometry visual mesh filename=package://my_robot/meshes/base_scan.STL
- link left_wheel_front_Link: geometry visual mesh filename=package://my_robot/meshes/left_wheel_front_Link.STL
- link left_wheel_rear_Link: geometry visual mesh filename=package://my_robot/meshes/left_wheel_rear_Link.STL
- link right_wheel_front_Link: geometry visual mesh filename=package://my_robot/meshes/right_wheel_front_Link.STL
- link right_wheel_rear_Link: geometry visual mesh filename=package://my_robot/meshes/right_wheel_rear_Link.STL

Commit message: update 2026-06-26 16:26:35

File: ros_motion_planning/my_robot/urdf/my_robot.urdf (robot description, URDF)
Before this commit: robot my_robot, 6 links, 5 joints
Links:
- link base_link: geometry collision mesh filename=package://my_robot/meshes/base_link.STL; visual mesh filename=package://my_robot/meshes/base_link.STL
- link base_scan: geometry collision mesh filename=package://my_robot/meshes/base_scan.STL; visual mesh filename=package://my_robot/meshes/base_scan.STL
- link left_wheel_front_Link: geometry collision mesh filename=package://my_robot/meshes/left_wheel_front_Link.STL; visual mesh filename=package://my_robot/meshes/left_wheel_front_Link.STL
- link left_wheel_rear_Link: geometry collision mesh filename=package://my_robot/meshes/left_wheel_rear_Link.STL; visual mesh filename=package://my_robot/meshes/left_wheel_rear_Link.STL
- link right_wheel_front_Link: geometry collision mesh filename=package://my_robot/meshes/right_wheel_front_Link.STL; visual mesh filename=package://my_robot/meshes/right_wheel_front_Link.STL
- link right_wheel_rear_Link: geometry collision mesh filename=package://my_robot/meshes/right_wheel_rear_Link.STL; visual mesh filename=package://my_robot/meshes/right_wheel_rear_Link.STL

Commit message: update 2026-06-26 16:49:59

File: ros_motion_planning/my_robot/urdf/my_robot.urdf (robot description, URDF)
Before this commit: robot my_robot, 6 links, 5 joints
Joints:
- joint left_wheel_front_joint: type continuous -> fixed
- joint left_wheel_rear_joint: type continuous -> fixed
- joint right_wheel_front_joint: type continuous -> fixed
- joint right_wheel_rear_joint: type continuous -> fixed

Commit message: update 2026-06-26 17:32:19

File: ros_motion_planning/my_robot/urdf/my_robot.urdf (robot description, URDF)
Before this commit: robot my_robot, 6 links, 5 joints
Links:
- link base_link: geometry collision box size=0.5 0.3 0.15; visual box size=0.5 0.3 0.15
- link base_scan: geometry collision cylinder length=0.06 radius=0.04; visual cylinder length=0.06 radius=0.04
- link left_wheel_front_Link: geometry collision cylinder length=0.035 radius=0.07; visual cylinder length=0.035 radius=0.07
- link left_wheel_rear_Link: geometry collision cylinder length=0.035 radius=0.07; visual cylinder length=0.035 radius=0.07
- link right_wheel_front_Link: geometry collision cylinder length=0.035 radius=0.07; visual cylinder length=0.035 radius=0.07
- link right_wheel_rear_Link: geometry collision cylinder length=0.035 radius=0.07; visual cylinder length=0.035 radius=0.07
Joints:
- joint left_wheel_front_joint: origin xyz=0.178912109148856 0.107037805223412 0.030052752271374 rpy=0 0 0 -> xyz=0.178912109148856 0.107037805223412 0.030052752271374 rpy=1.5708 0 0
- joint left_wheel_rear_joint: origin xyz=-0.157035966824235 0.101175564800452 0.0300400994124252 rpy=0 0 0 -> xyz=-0.157035966824235 0.101175564800452 0.0300400994124252 rpy=1.5708 0 0
- joint right_wheel_front_joint: origin xyz=0.181032384121442 -0.10075683114026 0.0299585988024258 rpy=0 0 0 -> xyz=0.181032384121442 -0.10075683114026 0.0299585988024258 rpy=1.5708 0 0

Commit message: update 2026-06-26 17:34:29

File: ros_motion_planning/my_robot/urdf/my_robot.urdf (robot description, URDF)
Before this commit: robot my_robot, 6 links, 5 joints
Links:
- link base_link: geometry collision mesh filename=package://my_robot/meshes/base_link.STL; visual mesh filename=package://my_robot/meshes/base_link.STL
- link base_scan: geometry collision mesh filename=package://my_robot/meshes/base_scan.STL; visual mesh filename=package://my_robot/meshes/base_scan.STL
- link left_wheel_front_Link: geometry collision mesh filename=package://my_robot/meshes/left_wheel_front_Link.STL; visual mesh filename=package://my_robot/meshes/left_wheel_front_Link.STL
- link left_wheel_rear_Link: geometry collision mesh filename=package://my_robot/meshes/left_wheel_rear_Link.STL; visual mesh filename=package://my_robot/meshes/left_wheel_rear_Link.STL
- link right_wheel_front_Link: geometry collision mesh filename=package://my_robot/meshes/right_wheel_front_Link.STL; visual mesh filename=package://my_robot/meshes/right_wheel_front_Link.STL
- link right_wheel_rear_Link: geometry collision mesh filename=package://my_robot/meshes/right_wheel_rear_Link.STL; visual mesh filename=package://my_robot/meshes/right_wheel_rear_Link.STL
Joints:
- joint left_wheel_front_joint: origin xyz=0.178912109148856 0.107037805223412 0.030052752271374 rpy=1.5708 0 0 -> xyz=0.178912109148856 0.107037805223412 0.030052752271374 rpy=0 0 0
- joint left_wheel_rear_joint: origin xyz=-0.157035966824235 0.101175564800452 0.0300400994124252 rpy=1.5708 0 0 -> xyz=-0.157035966824235 0.101175564800452 0.0300400994124252 rpy=0 0 0
- joint right_wheel_front_joint: origin xyz=0.181032384121442 -0.10075683114026 0.0299585988024258 rpy=1.5708 0 0 -> xyz=0.181032384121442 -0.10075683114026 0.0299585988024258 rpy=0 0 0
