Commit message: update 2026-10-09 19:13:31

File: new_robot/urdf/new_robot.urdf (robot description, URDF)
Before this commit: robot new_robot, 6 links, 5 joints
Links:
- added link base_footprint
Joints:
- added joint base_footprint_joint: type fixed, parent base_footprint, child base_link, origin xyz=0 0 0 rpy=0 0 -0.01989

Commit message: update 2026-10-09 19:31:58

File: new_robot/urdf/new_robot.urdf (robot description, URDF)
Before this commit: robot new_robot, 7 links, 6 joints
Links:
- removed link base_footprint
- link base_link: mass 4.24802348273642 -> 1.95161426437595
- link base_scan: mass 0.0374307368945306 -> 0.037430736894531
- link left_wheel_rear_Link: mass 0.826148513927946 -> 0.826148513927947
- link right_wheel_front_Link: mass 0.826148516893895 -> 0.826148516893894
Joints:
- removed joint base_footprint_joint
- joint base_scan_joint: axis 0 0 0 -> 0 0 1; type fixed -> continuous

Commit message: update 2026-10-09 19:38:42

File: new_robot/urdf/new_robot.urdf (robot description, URDF)
Before this commit: robot new_robot, 6 links, 5 joints
Links:
- added link base_footprint
- link base_scan: geometry 
- link left_wheel_front_Link: geometry 
- link left_wheel_rear_Link: geometry 
- link right_wheel_front_Link: geometry 
- link right_wheel_rear_Link: geometry 
Joints:
- added joint base_footprint_joint: type fixed, parent base_footprint, child base_link, origin xyz=0 0 0 rpy=0 0 -0.01989
- joint base_scan_joint: axis 0 0 1 -> (none); type continuous -> fixed
